Commit message: pre_outdoor_2

File: src/quadrotor_description/urdf/quadrotor_ros.urdf (robot description, URDF)
Before this commit: robot quadrotor, 5 links, 4 joints
Links:
- removed link laser0_frame
- added link hokuyo_frame, mass 0.270; collision box size=0.058 0.058 0.087; visual mesh filename=package://hector_sensors_description/meshes/hokuyo_utm30lx/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
Joints:
- joint laser0_joint: child laser0_frame -> hokuyo_frame
